Commit message: add inertia

File: description/omnibot.urdf.xacro (robot description, xacro)
@@ -1,4 +1,5 @@
 <?xml version="1.0"?>
-<robot name="omnibot">
+<robot xmlns:xacro="http://www.ros.org/wiki/xacro" name="omnibot">
+	<xacro:include filename="inertial_macros.xacro"/>
 	<link name="base_link">
 		<visual>
@@ -11,4 +12,13 @@
 			</material>
 		</visual>
+		<collision>
+			<geometry>
+				<box size="0.326 0.206 .094"/>
+			</geometry>
+			<origin xyz="0 0 0.072"/>
+		</collision>
+		<xacro:inertial_box mass="0.5" x="0.326" y="0.206" z="0.094">
+			<origin xyz="0 0 0.072"/>
+		</xacro:inertial_box>
 	</link>
 	<link name="base_laser">

Commit message: adding planar controller

File: description/omnibot.urdf.xacro (robot description, xacro)
@@ -2,4 +2,5 @@
 <robot xmlns:xacro="http://www.ros.org/wiki/xacro" name="omnibot">
 	<xacro:include filename="inertial_macros.xacro"/>
+	<xacro:include filename="gazebo_control.xacro"/>
 	<link name="base_link">
 		<visual>
@@ -28,4 +29,12 @@
 			</geometry>
 		</visual>
+		<collision>
+			<geometry>
+				<cylinder length="0.02" radius="0.04"/>
+			</geometry>
+		</collision>
+		<xacro:inertial_cylinder mass="0.1" length="0.02" radius="0.04">
+			<origin xyz="0 0 0"/>
+		</xacro:inertial_cylinder>
 	</link>
 	<joint name="base_link_to_base_laser" type="fixed">
@@ -34,3 +43,9 @@
 		<origin rpy="0 0 -0.05" xyz="0.097 0.0 0.125"/>
 	</joint>
+	<gazebo reference="base_link">
+		<material>Gazebo/Red</material>
+	</gazebo>
+	<gazebo reference="base_laser">
+		<material>Gazebo/Blue</material>
+	</gazebo>
 </robot>

Commit message: configuring the lidar plugin for gazebo

File: description/omnibot.urdf.xacro (robot description, xacro)
@@ -32,5 +32,35 @@
 		<parent link="base_link"/>
 		<child link="base_laser"/>
-		<origin rpy="0 0 -0.05" xyz="0.097 0.0 0.125"/>
+		<origin rpy="0 0 0" xyz="0.097 0.0 0.125"/>
 	</joint>
+	<gazebo reference="base_laser">
+		<material>Gazebo/Red</material>
+		<sensor type="ray" name="base_laser">
+			<pose>0 0 0 0 0 0</pose>
+			<visualize>true</visualize>
+			<update_rate>10</update_rate>
+			<ray>
+				<scan>
+					<horizontal>
+						<samples>360</samples>
+						<resolution>1</resolution>
+						<min_angle>-3.1415926535897931</min_angle>
+						<max_angle>3.1415926535897931</max_angle>
+					</horizontal>
+				</scan>
+				<range>
+					<min>0.3</min>
+					<max>12</max>
+					<resolution>0.01</resolution>
+				</range>
+			</ray>
+			<plugin name="base_laser_controller" filename="libgazebo_ros_ray_sensor.so">
+				<ros>
+					<argument>~/out:=scan</argument>
+				</ros>
+				<output_type>sensor_msgs/LaserScan</output_type>
+				<frameName>base_laser</frameName>
+			</plugin>
+		</sensor>
+	</gazebo>
 </robot>

Commit message: better launch and test script

File: description/omnibot.urdf.xacro (robot description, xacro)
@@ -6,5 +6,5 @@
 		<visual>
 			<geometry>
-				<box size="0.326 0.206 .094"/>
+				<box size="0.26 0.25 0.14"/>
 			</geometry>
 			<origin xyz="0 0 0.072"/>
@@ -15,5 +15,5 @@
 		<collision>
 			<geometry>
-				<box size="0.326 0.206 .094"/>
+				<box size="0.26 0.25 0.14"/>
 			</geometry>
 			<origin xyz="0 0 0.072"/>
@@ -26,10 +26,10 @@
 		<visual>
 			<geometry>
-				<cylinder length="0.02" radius="0.04"/>
+				<cylinder length="0.027" radius="0.035"/>
 			</geometry>
 		</visual>
 		<collision>
 			<geometry>
-				<cylinder length="0.02" radius="0.04"/>
+				<cylinder length="0.027" radius="0.035"/>
 			</geometry>
 		</collision>
@@ -41,5 +41,5 @@
 		<parent link="base_link"/>
 		<child link="base_laser"/>
-		<origin rpy="0 0 0" xyz="0.097 0.0 0.125"/>
+		<origin rpy="0 0 0" xyz="0.075 0 0.1535"/>
 	</joint>
 	<gazebo reference="base_laser">

Commit message: updating lidar pos

File: description/omnibot.urdf.xacro (robot description, xacro)
@@ -41,5 +41,6 @@
 		<parent link="base_link"/>
 		<child link="base_laser"/>
-		<origin rpy="0 0 0" xyz="0.075 0 0.1535"/>
+		<origin rpy="0 0 0" xyz="0 0 0.1535"/>
+		<!-- <origin rpy="0 0 0" xyz="0.075 0 0.1535"/> -->
 	</joint>
 	<gazebo reference="base_laser">
@@ -59,5 +60,5 @@
 				</scan>
 				<range>
-					<min>0.3</min>
+					<min>0.15</min>
 					<max>12</max>
 					<resolution>0.01</resolution>
